File: tmc2660/tmc2660-block-100.sch (KiCad schematic (older format))
At the start: 18 parts, among them J100 0R, M100 Mount, M101 Mount, P100 Motor, U100 TMC2660

Commit message: Finished squished board
Parts:
- removed M100: Mount, Mounting_Holes:MountingHole_2.7mm_M2.5, symbol Mechanical:Mounting_Hole
- removed M101: Mount, Mounting_Holes:MountingHole_2.7mm_M2.5_Pad, symbol Mechanical:Mounting_Hole_PAD
Connections:
- net labels added: STALL
- wire segments 63 -> 64
- no-connect marks 2 -> 1
Changed lines of the file:
@@
 EESchema Schematic File Version 4
+LIBS:tmc2660-quad-cache
 EELAYER 26 0
 EELAYER END
 $Descr A4 11693 8268
 encoding utf-8
-Sheet 2 2
+Sheet 2 5
 Title ""
 Date ""
@@
 $Comp
 L device:C C103
-U 1 1 5A0CA5B9
+U 1 1 5A369CD8
 P 4400 2300
 F 0 "C103" H 4425 2400 50  0000 L CNN
@@
 $Comp
 L device:C C102
-U 1 1 5A0CA5C0
+U 1 1 5A369CDB
 P 4100 2300
 F 0 "C102" H 4125 2400 50  0000 L CNN
@@
 $Comp
 L power:GND #PWR0101
-U 1 1 5A0CA5C7
+U 1 1 5A369CDE
 P 3800 3050
 F 0 "#PWR0101" H 3800 2800 50  0001 C CNN
@@
 $Comp
 L power:GND #PWR0102
-U 1 1 5A0CA5CD
+U 1 1 5A369CE1
 P 4400 2450
 F 0 "#PWR0102" H 4400 2200 50  0001 C CNN
@@
 $Comp
 L device:C C104
-U 1 1 5A0CA5D3
+U 1 1 5A369CE4
 P 2900 1700
 F 0 "C104" H 2800 2000 50  0000 L CNN
@@
 $Comp
 L device:C C105
-U 1 1 5A0CA5DE
+U 1 1 5A369CE7
 P 3200 1700
 F 0 "C105" H 3150 2000 50  0000 L CNN
@@
 $Comp
 L power:GND #PWR0103
-U 1 1 5A0CA5E6
+U 1 1 5A369CEA
 P 3350 1850
 F 0 "#PWR0103" H 3350 1600 50  0001 C CNN
@@
 $Comp
 L power:GND #PWR0104
-U 1 1 5A0CA5EF
+U 1 1 5A369CEC
 P 2800 3800
 F 0 "#PWR0104" H 2800 3550 50  0001 C CNN
@@
 $Comp
 L device:R R102
-U 1 1 5A0CA5FF
+U 1 1 5A369CF3
 P 3950 3550
 F 0 "R102" V 3850 3550 50  0000 C CNN
@@
 $Comp
 L Connector:Conn_01x04 P100
-U 1 1 5A0CA611
+U 1 1 5A369CF9
 P 5150 2950
 F 0 "P100" H 5150 3200 50  0000 C CNN
@@
 $Comp
 L device:C C108
-U 1 1 5A0CA61C
+U 1 1 5A369CFC
 P 2200 3400
 F 0 "C108" H 2225 3500 50  0000 L CNN
@@
 $Comp
 L tmc2660:TMC2660 U100
-U 1 1 5A0CA62A
+U 1 1 5A369D03
 P 2950 2850
 F 0 "U100" H 2950 3150 60  0000 C CNN
@@
 $Comp
 L device:C C106
-U 1 1 5A0CA648
+U 1 1 5A369D08
 P 2250 3700
 F 0 "C106" H 1950 3700 50  0000 L CNN
@@
 $Comp
 L device:C_Small C101
-U 1 1 5A0CA67B
+U 1 1 5A369D17
 P 3800 2950
 F 0 "C101" H 3900 3000 50  0000 L CNN
@@
 $Comp
 L device:C_Small C100
-U 1 1 5A0CA683
+U 1 1 5A369D19
 P 3750 3850
 F 0 "C100" H 3450 3800 50  0000 L CNN
@@
 Text Label 3500 2800 0    40   ~ 0
 BRA
-NoConn ~ 2350 3150
 Text Label 2000 2850 0    60   ~ 0
 STEP
@@
 $Comp
 L device:R J100
-U 1 1 5A0CA6C8
+U 1 1 5A369D1F
 P 1450 2350
 F 0 "J100" H 1550 2500 50  0000 C CNN
@@
 Text Label 4800 3150 0    60   ~ 0
 B2
-$Comp
-L Mechanical:Mounting_Hole M100
-U 1 1 5A0FBC47
-P 1250 4250
-F 0 "M100" H 1150 4400 50  0000 L CNN
-F 1 "Mount" H 1308 4279 50  0000 L CNN
-F 2 "Mounting_Holes:MountingHole_2.7mm_M2.5" H 1450 4250 50  0001 C CNN
-F 3 "~" H 1450 4250 50  0001 C CNN
-	1    1250 4250
-	1    0    0    -1
-$EndComp
-$Comp
-L Mechanical:Mounting_Hole_PAD M101
-U 1 1 5A0FBD0F
-P 1650 4300
-F 0 "M101" H 1550 4500 50  0000 L CNN
-F 1 "Mount" H 1708 4329 50  0000 L CNN
-F 2 "Mounting_Holes:MountingHole_2.7mm_M2.5_Pad" H 1850 4300 50  0001 C CNN
-F 3 "~" H 1850 4300 50  0001 C CNN
-	1    1650 4300
-	1    0    0    -1
-$EndComp
 Wire Wire Line
 	3050 1550 3050 1950
@@
 $Comp
 L power:GND #PWR01
-U 1 1 5A17CB15
+U 1 1 5A369D24
 P 4600 3200
 F 0 "#PWR01" H 4600 2950 50  0001 C CNN
@@
 Text Notes 4500 3750 0    51   ~ 0
 Sense Resistors alternatively\nalso with 100mOhm
-$Comp
-L power:GND #PWR?
-U 1 1 5A1C342B
-P 1650 4400
-F 0 "#PWR?" H 1650 4150 50  0001 C CNN
-F 1 "GND" H 1650 4250 50  0000 C CNN
-F 2 "" H 1650 4400 60  0000 C CNN
-F 3 "" H 1650 4400 60  0000 C CNN
-	1    1650 4400
-	1    0    0    -1
-$EndComp
 Wire Wire Line
 	3050 1550 3200 1550
@@
 Wire Wire Line
 	3750 3550 3800 3550
+Text HLabel 1950 3150 0    60   Output ~ 0
+STALL
+Wire Wire Line
+	1950 3150 2350 3150
+Text Label 2000 3150 0    60   ~ 0
+STALL
 $EndSCHEMATC
