File: tmc2660/tmc2660-block-200.sch (KiCad schematic (older format))
At the start: 18 parts, among them J200 0R, M200 Mount, M201 Mount, P200 Motor, U200 TMC2660

Commit message: Finished squished board
Parts:
- removed M200: Mount, Mounting_Holes:MountingHole_2.7mm_M2.5, symbol Mechanical:Mounting_Hole
- removed M201: Mount, Mounting_Holes:MountingHole_2.7mm_M2.5_Pad, symbol Mechanical:Mounting_Hole_PAD
Connections:
- net labels added: STALL
- wire segments 63 -> 64
- no-connect marks 2 -> 1
Changed lines of the file:
@@
 EESchema Schematic File Version 4
+LIBS:tmc2660-quad-cache
 EELAYER 26 0
 EELAYER END
 $Descr A4 11693 8268
 encoding utf-8
-Sheet 2 2
+Sheet 5 5
 Title ""
 Date ""
@@
 $Comp
 L device:C C203
-U 1 1 5A0CA5B9
+U 1 1 5A369CD7
 P 4400 2300
 F 0 "C203" H 4425 2400 50  0000 L CNN
@@
 $Comp
 L device:C C202
-U 1 1 5A0CA5C0
+U 1 1 5A369CDA
 P 4100 2300
 F 0 "C202" H 4125 2400 50  0000 L CNN
@@
 $EndComp
 $Comp
-L power:GND #PWR0101
-U 1 1 5A0CA5C7
+L power:GND #PWR023
+U 1 1 5A369CDD
 P 3800 3050
-F 0 "#PWR0101" H 3800 2800 50  0001 C CNN
+F 0 "#PWR023" H 3800 2800 50  0001 C CNN
 F 1 "GND" H 3800 2900 50  0000 C CNN
 F 2 "" H 3800 3050 60  0000 C CNN
@@
 $EndComp
 $Comp
-L power:GND #PWR0102
-U 1 1 5A0CA5CD
+L power:GND #PWR024
+U 1 1 5A369CE0
 P 4400 2450
-F 0 "#PWR0102" H 4400 2200 50  0001 C CNN
+F 0 "#PWR024" H 4400 2200 50  0001 C CNN
 F 1 "GND" H 4400 2300 50  0000 C CNN
 F 2 "" H 4400 2450 60  0000 C CNN
@@
 $Comp
 L device:C C205
-U 1 1 5A0CA5DE
+U 1 1 5A369CE6
 P 3200 1700
 F 0 "C205" H 3150 2000 50  0000 L CNN
@@
 $EndComp
 $Comp
-L power:GND #PWR0103
-U 1 1 5A0CA5E6
+L power:GND #PWR025
+U 1 1 5A369CE9
 P 3350 1850
-F 0 "#PWR0103" H 3350 1600 50  0001 C CNN
+F 0 "#PWR025" H 3350 1600 50  0001 C CNN
 F 1 "GND" H 3450 1750 50  0000 C CNN
 F 2 "" H 3350 1850 60  0000 C CNN
@@
 $EndComp
 $Comp
-L power:GND #PWR0104
+L power:GND #PWR026
 U 1 1 5A0CA5EF
 P 2800 3800
-F 0 "#PWR0104" H 2800 3550 50  0001 C CNN
+F 0 "#PWR026" H 2800 3550 50  0001 C CNN
 F 1 "GND" H 2800 3650 50  0000 C CNN
 F 2 "" H 2800 3800 60  0000 C CNN
@@
 $Comp
 L device:R R203
-U 1 1 5A0CA5F8
+U 1 1 5A369CEF
 P 3950 2700
 F 0 "R203" V 4050 2700 50  0000 C CNN
@@
 $EndComp
 $Comp
-L power:GND #PWR0105
-U 1 1 5A0CA606
+L power:GND #PWR027
+U 1 1 5A369CF6
 P 3750 3950
-F 0 "#PWR0105" H 3750 3700 50  0001 C CNN
+F 0 "#PWR027" H 3750 3700 50  0001 C CNN
 F 1 "GND" H 3750 3800 50  0000 C CNN
 F 2 "" H 3750 3950 60  0000 C CNN
@@
 $Comp
 L Connector:Conn_01x04 P200
-U 1 1 5A0CA611
+U 1 1 5A369CFA
 P 5150 2950
 F 0 "P200" H 5150 3200 50  0000 C CNN
@@
 $EndComp
 $Comp
-L power:GND #PWR0106
-U 1 1 5A0CA623
+L power:GND #PWR028
+U 1 1 5A369CFF
 P 2050 3400
-F 0 "#PWR0106" H 2050 3150 50  0001 C CNN
+F 0 "#PWR028" H 2050 3150 50  0001 C CNN
 F 1 "GND" H 2050 3250 50  0000 C CNN
 F 2 "" H 2050 3400 60  0000 C CNN
@@
 $Comp
 L tmc2660:TMC2660 U200
-U 1 1 5A0CA62A
+U 1 1 5A369D01
 P 2950 2850
 F 0 "U200" H 2950 3150 60  0000 C CNN
@@
 $EndComp
 $Comp
-L power:GND #PWR0107
-U 1 1 5A0CA642
+L power:GND #PWR029
+U 1 1 5A369D05
 P 2250 3850
-F 0 "#PWR0107" H 2250 3600 50  0001 C CNN
+F 0 "#PWR029" H 2250 3600 50  0001 C CNN
 F 1 "GND" H 2250 3700 50  0000 C CNN
 F 2 "" H 2250 3850 60  0000 C CNN
@@
 $Comp
 L device:C C206
-U 1 1 5A0CA648
+U 1 1 5A369D09
 P 2250 3700
 F 0 "C206" H 1950 3700 50  0000 L CNN
@@
 NoConn ~ 2350 3250
 $Comp
-L power:GND #PWR0108
-U 1 1 5A0CA65B
+L power:GND #PWR030
+U 1 1 5A369D0B
 P 2250 2250
-F 0 "#PWR0108" H 2250 2000 50  0001 C CNN
+F 0 "#PWR030" H 2250 2000 50  0001 C CNN
 F 1 "GND" H 2250 2100 50  0000 C CNN
 F 2 "" H 2250 2250 60  0000 C CNN
@@
 $EndComp
 $Comp
-L power:GND #PWR0109
-U 1 1 5A0CA666
+L power:GND #PWR031
+U 1 1 5A369D0E
 P 2500 3800
-F 0 "#PWR0109" H 2500 3550 50  0001 C CNN
+F 0 "#PWR031" H 2500 3550 50  0001 C CNN
 F 1 "GND" H 2450 3650 50  0000 C CNN
 F 2 "" H 2500 3800 60  0000 C CNN
@@
 $Comp
 L device:R R200
-U 1 1 5A0CA66C
+U 1 1 5A369D11
 P 4400 3500
 F 0 "R200" H 4200 3500 50  0000 C CNN
@@
 $Comp
 L device:R R201
-U 1 1 5A0CA673
+U 1 1 5A369D14
 P 4400 2950
 F 0 "R201" H 4600 2900 50  0000 C CNN
@@
 $Comp
 L device:C_Small C201
-U 1 1 5A0CA67B
+U 1 1 5A369D16
 P 3800 2950
 F 0 "C201" H 3900 3000 50  0000 L CNN
@@
 $Comp
 L device:C_Small C200
-U 1 1 5A0CA683
+U 1 1 5A369D1A
 P 3750 3850
 F 0 "C200" H 3450 3800 50  0000 L CNN
@@
 Text Label 3500 2800 0    40   ~ 0
 BRA
-NoConn ~ 2350 3150
 Text Label 2000 2850 0    60   ~ 0
 STEP
@@
 $Comp
 L device:CP C207
-U 1 1 5A0CA6BD
+U 1 1 5A369D1E
 P 3500 1700
 F 0 "C207" H 3450 2000 50  0000 L CNN
@@
 Text Label 4800 3150 0    60   ~ 0
 B2
-$Comp
-L Mechanical:Mounting_Hole M200
-U 1 1 5A0FBC47
-P 1250 4250
-F 0 "M200" H 1150 4400 50  0000 L CNN
-F 1 "Mount" H 1308 4279 50  0000 L CNN
-F 2 "Mounting_Holes:MountingHole_2.7mm_M2.5" H 1450 4250 50  0001 C CNN
-F 3 "~" H 1450 4250 50  0001 C CNN
-	1    1250 4250
-	1    0    0    -1
-$EndComp
-$Comp
-L Mechanical:Mounting_Hole_PAD M201
-U 1 1 5A0FBD0F
-P 1650 4300
-F 0 "M201" H 1550 4500 50  0000 L CNN
-F 1 "Mount" H 1708 4329 50  0000 L CNN
-F 2 "Mounting_Holes:MountingHole_2.7mm_M2.5_Pad" H 1850 4300 50  0001 C CNN
-F 3 "~" H 1850 4300 50  0001 C CNN
-	1    1650 4300
-	1    0    0    -1
-$EndComp
 Wire Wire Line
 	3050 1550 3050 1950
@@
 Connection ~ 4250 2800
 $Comp
-L power:GND #PWR01
-U 1 1 5A17CB15
+L power:GND #PWR032
+U 1 1 5A369D23
 P 4600 3200
-F 0 "#PWR01" H 4600 2950 50  0001 C CNN
+F 0 "#PWR032" H 4600 2950 50  0001 C CNN
 F 1 "GND" H 4600 3050 50  0000 C CNN
 F 2 "" H 4600 3200 60  0000 C CNN
@@
 Sense Resistors alternatively\nalso with 100mOhm
 $Comp
-L power:GND #PWR?
+L power:GND #PWR033
 U 1 1 5A1C342B
 P 1650 4400
-F 0 "#PWR?" H 1650 4150 50  0001 C CNN
+F 0 "#PWR033" H 1650 4150 50  0001 C CNN
 F 1 "GND" H 1650 4250 50  0000 C CNN
 F 2 "" H 1650 4400 60  0000 C CNN
@@
 Wire Wire Line
 	3750 3550 3800 3550
+Text HLabel 1950 3150 0    60   Output ~ 0
+STALL
+Wire Wire Line
+	1950 3150 2350 3150
+Text Label 2000 3150 0    60   ~ 0
+STALL
 $EndSCHEMATC
