File: tmc2660/tmc2660-block-300.sch (KiCad schematic (older format))
At the start: 18 parts, among them J300 0R, M300 Mount, M301 Mount, P300 Motor, U300 TMC2660

Commit message: Finished squished board
Parts:
- removed M300: Mount, Mounting_Holes:MountingHole_2.7mm_M2.5, symbol Mechanical:Mounting_Hole
- removed M301: Mount, Mounting_Holes:MountingHole_2.7mm_M2.5_Pad, symbol Mechanical:Mounting_Hole_PAD
Connections:
- net labels added: STALL
- wire segments 63 -> 64
- no-connect marks 2 -> 1
Changed lines of the file:
@@
 EESchema Schematic File Version 4
+LIBS:tmc2660-quad-cache
 EELAYER 26 0
 EELAYER END
 $Descr A4 11693 8268
 encoding utf-8
-Sheet 2 2
+Sheet 3 5
 Title ""
 Date ""
@@
 $Comp
 L device:C C303
-U 1 1 5A0CA5B9
+U 1 1 5A369CD9
 P 4400 2300
 F 0 "C303" H 4425 2400 50  0000 L CNN
@@
 $EndComp
 $Comp
-L power:GND #PWR0101
+L power:GND #PWR03
 U 1 1 5A0CA5C7
 P 3800 3050
-F 0 "#PWR0101" H 3800 2800 50  0001 C CNN
+F 0 "#PWR03" H 3800 2800 50  0001 C CNN
 F 1 "GND" H 3800 2900 50  0000 C CNN
 F 2 "" H 3800 3050 60  0000 C CNN
@@
 $EndComp
 $Comp
-L power:GND #PWR0102
-U 1 1 5A0CA5CD
+L power:GND #PWR04
+U 1 1 5A369CE2
 P 4400 2450
-F 0 "#PWR0102" H 4400 2200 50  0001 C CNN
+F 0 "#PWR04" H 4400 2200 50  0001 C CNN
 F 1 "GND" H 4400 2300 50  0000 C CNN
 F 2 "" H 4400 2450 60  0000 C CNN
@@
 $Comp
 L device:C C304
-U 1 1 5A0CA5D3
+U 1 1 5A369CE3
 P 2900 1700
 F 0 "C304" H 2800 2000 50  0000 L CNN
@@
 $EndComp
 $Comp
-L power:GND #PWR0103
-U 1 1 5A0CA5E6
+L power:GND #PWR05
+U 1 1 5A369CEB
 P 3350 1850
-F 0 "#PWR0103" H 3350 1600 50  0001 C CNN
+F 0 "#PWR05" H 3350 1600 50  0001 C CNN
 F 1 "GND" H 3450 1750 50  0000 C CNN
 F 2 "" H 3350 1850 60  0000 C CNN
@@
 $EndComp
 $Comp
-L power:GND #PWR0104
-U 1 1 5A0CA5EF
+L power:GND #PWR06
+U 1 1 5A369CED
 P 2800 3800
-F 0 "#PWR0104" H 2800 3550 50  0001 C CNN
+F 0 "#PWR06" H 2800 3550 50  0001 C CNN
 F 1 "GND" H 2800 3650 50  0000 C CNN
 F 2 "" H 2800 3800 60  0000 C CNN
@@
 $Comp
 L device:R R303
-U 1 1 5A0CA5F8
+U 1 1 5A369CF0
 P 3950 2700
 F 0 "R303" V 4050 2700 50  0000 C CNN
@@
 $Comp
 L device:R R302
-U 1 1 5A0CA5FF
+U 1 1 5A369CF2
 P 3950 3550
 F 0 "R302" V 3850 3550 50  0000 C CNN
@@
 $EndComp
 $Comp
-L power:GND #PWR0105
-U 1 1 5A0CA606
+L power:GND #PWR07
+U 1 1 5A369CF5
 P 3750 3950
-F 0 "#PWR0105" H 3750 3700 50  0001 C CNN
+F 0 "#PWR07" H 3750 3700 50  0001 C CNN
 F 1 "GND" H 3750 3800 50  0000 C CNN
 F 2 "" H 3750 3950 60  0000 C CNN
@@
 $Comp
 L device:C C308
-U 1 1 5A0CA61C
+U 1 1 5A369CFD
 P 2200 3400
 F 0 "C308" H 2225 3500 50  0000 L CNN
@@
 $EndComp
 $Comp
-L power:GND #PWR0106
-U 1 1 5A0CA623
+L power:GND #PWR08
+U 1 1 5A369D00
 P 2050 3400
-F 0 "#PWR0106" H 2050 3150 50  0001 C CNN
+F 0 "#PWR08" H 2050 3150 50  0001 C CNN
 F 1 "GND" H 2050 3250 50  0000 C CNN
 F 2 "" H 2050 3400 60  0000 C CNN
@@
 $EndComp
 $Comp
-L power:GND #PWR0107
-U 1 1 5A0CA642
+L power:GND #PWR09
+U 1 1 5A369D04
 P 2250 3850
-F 0 "#PWR0107" H 2250 3600 50  0001 C CNN
+F 0 "#PWR09" H 2250 3600 50  0001 C CNN
 F 1 "GND" H 2250 3700 50  0000 C CNN
 F 2 "" H 2250 3850 60  0000 C CNN
@@
 $Comp
 L device:C C306
-U 1 1 5A0CA648
+U 1 1 5A369D07
 P 2250 3700
 F 0 "C306" H 1950 3700 50  0000 L CNN
@@
 NoConn ~ 2350 3250
 $Comp
-L power:GND #PWR0108
-U 1 1 5A0CA65B
+L power:GND #PWR010
+U 1 1 5A369D0A
 P 2250 2250
-F 0 "#PWR0108" H 2250 2000 50  0001 C CNN
+F 0 "#PWR010" H 2250 2000 50  0001 C CNN
 F 1 "GND" H 2250 2100 50  0000 C CNN
 F 2 "" H 2250 2250 60  0000 C CNN
@@
 $EndComp
 $Comp
-L power:GND #PWR0109
-U 1 1 5A0CA666
+L power:GND #PWR011
+U 1 1 5A369D0F
 P 2500 3800
-F 0 "#PWR0109" H 2500 3550 50  0001 C CNN
+F 0 "#PWR011" H 2500 3550 50  0001 C CNN
 F 1 "GND" H 2450 3650 50  0000 C CNN
 F 2 "" H 2500 3800 60  0000 C CNN
@@
 $Comp
 L device:R R300
-U 1 1 5A0CA66C
+U 1 1 5A369D12
 P 4400 3500
 F 0 "R300" H 4200 3500 50  0000 C CNN
@@
 $Comp
 L device:R R301
-U 1 1 5A0CA673
+U 1 1 5A369D15
 P 4400 2950
 F 0 "R301" H 4600 2900 50  0000 C CNN
@@
 $Comp
 L device:C_Small C300
-U 1 1 5A0CA683
+U 1 1 5A369D1B
 P 3750 3850
 F 0 "C300" H 3450 3800 50  0000 L CNN
@@
 Text Label 3500 2800 0    40   ~ 0
 BRA
-NoConn ~ 2350 3150
 Text Label 2000 2850 0    60   ~ 0
 STEP
@@
 $Comp
 L device:CP C307
-U 1 1 5A0CA6BD
+U 1 1 5A369D1D
 P 3500 1700
 F 0 "C307" H 3450 2000 50  0000 L CNN
@@
 $Comp
 L device:R J300
-U 1 1 5A0CA6C8
+U 1 1 5A369D21
 P 1450 2350
 F 0 "J300" H 1550 2500 50  0000 C CNN
@@
 Text Label 4800 3150 0    60   ~ 0
 B2
-$Comp
-L Mechanical:Mounting_Hole M300
-U 1 1 5A0FBC47
-P 1250 4250
-F 0 "M300" H 1150 4400 50  0000 L CNN
-F 1 "Mount" H 1308 4279 50  0000 L CNN
-F 2 "Mounting_Holes:MountingHole_2.7mm_M2.5" H 1450 4250 50  0001 C CNN
-F 3 "~" H 1450 4250 50  0001 C CNN
-	1    1250 4250
-	1    0    0    -1
-$EndComp
-$Comp
-L Mechanical:Mounting_Hole_PAD M301
-U 1 1 5A0FBD0F
-P 1650 4300
-F 0 "M301" H 1550 4500 50  0000 L CNN
-F 1 "Mount" H 1708 4329 50  0000 L CNN
-F 2 "Mounting_Holes:MountingHole_2.7mm_M2.5_Pad" H 1850 4300 50  0001 C CNN
-F 3 "~" H 1850 4300 50  0001 C CNN
-	1    1650 4300
-	1    0    0    -1
-$EndComp
 Wire Wire Line
 	3050 1550 3050 1950
@@
 Connection ~ 4250 2800
 $Comp
-L power:GND #PWR01
-U 1 1 5A17CB15
+L power:GND #PWR012
+U 1 1 5A369D22
 P 4600 3200
-F 0 "#PWR01" H 4600 2950 50  0001 C CNN
+F 0 "#PWR012" H 4600 2950 50  0001 C CNN
 F 1 "GND" H 4600 3050 50  0000 C CNN
 F 2 "" H 4600 3200 60  0000 C CNN
@@
 Text Notes 4500 3750 0    51   ~ 0
 Sense Resistors alternatively\nalso with 100mOhm
-$Comp
-L power:GND #PWR?
-U 1 1 5A1C342B
-P 1650 4400
-F 0 "#PWR?" H 1650 4150 50  0001 C CNN
-F 1 "GND" H 1650 4250 50  0000 C CNN
-F 2 "" H 1650 4400 60  0000 C CNN
-F 3 "" H 1650 4400 60  0000 C CNN
-	1    1650 4400
-	1    0    0    -1
-$EndComp
 Wire Wire Line
 	3050 1550 3200 1550
@@
 Wire Wire Line
 	3750 3550 3800 3550
+Text HLabel 1950 3150 0    60   Output ~ 0
+STALL
+Wire Wire Line
+	1950 3150 2350 3150
+Text Label 2000 3150 0    60   ~ 0
+STALL
 $EndSCHEMATC
