File: tmc2660/tmc2660-block-400.sch (KiCad schematic (older format))
At the start: 18 parts, among them J400 0R, M400 Mount, M401 Mount, P400 Motor, U400 TMC2660

Commit message: Finished squished board
Parts:
- removed M400: Mount, Mounting_Holes:MountingHole_2.7mm_M2.5, symbol Mechanical:Mounting_Hole
- removed M401: Mount, Mounting_Holes:MountingHole_2.7mm_M2.5_Pad, symbol Mechanical:Mounting_Hole_PAD
Connections:
- net labels added: STALL
- wire segments 63 -> 64
- no-connect marks 2 -> 1
Changed lines of the file:
@@
 EESchema Schematic File Version 4
+LIBS:tmc2660-quad-cache
 EELAYER 26 0
 EELAYER END
 $Descr A4 11693 8268
 encoding utf-8
-Sheet 2 2
+Sheet 4 5
 Title ""
 Date ""
@@
 $Comp
 L device:C C402
-U 1 1 5A0CA5C0
+U 1 1 5A369CDC
 P 4100 2300
 F 0 "C402" H 4125 2400 50  0000 L CNN
@@
 $EndComp
 $Comp
-L power:GND #PWR0101
-U 1 1 5A0CA5C7
+L power:GND #PWR013
+U 1 1 5A369CDF
 P 3800 3050
-F 0 "#PWR0101" H 3800 2800 50  0001 C CNN
+F 0 "#PWR013" H 3800 2800 50  0001 C CNN
 F 1 "GND" H 3800 2900 50  0000 C CNN
 F 2 "" H 3800 3050 60  0000 C CNN
@@
 $EndComp
 $Comp
-L power:GND #PWR0102
+L power:GND #PWR014
 U 1 1 5A0CA5CD
 P 4400 2450
-F 0 "#PWR0102" H 4400 2200 50  0001 C CNN
+F 0 "#PWR014" H 4400 2200 50  0001 C CNN
 F 1 "GND" H 4400 2300 50  0000 C CNN
 F 2 "" H 4400 2450 60  0000 C CNN
@@
 $Comp
 L device:C C404
-U 1 1 5A0CA5D3
+U 1 1 5A369CE5
 P 2900 1700
 F 0 "C404" H 2800 2000 50  0000 L CNN
@@
 $Comp
 L device:C C405
-U 1 1 5A0CA5DE
+U 1 1 5A369CE8
 P 3200 1700
 F 0 "C405" H 3150 2000 50  0000 L CNN
@@
 $EndComp
 $Comp
-L power:GND #PWR0103
+L power:GND #PWR015
 U 1 1 5A0CA5E6
 P 3350 1850
-F 0 "#PWR0103" H 3350 1600 50  0001 C CNN
+F 0 "#PWR015" H 3350 1600 50  0001 C CNN
 F 1 "GND" H 3450 1750 50  0000 C CNN
 F 2 "" H 3350 1850 60  0000 C CNN
@@
 $EndComp
 $Comp
-L power:GND #PWR0104
-U 1 1 5A0CA5EF
+L power:GND #PWR016
+U 1 1 5A369CEE
 P 2800 3800
-F 0 "#PWR0104" H 2800 3550 50  0001 C CNN
+F 0 "#PWR016" H 2800 3550 50  0001 C CNN
 F 1 "GND" H 2800 3650 50  0000 C CNN
 F 2 "" H 2800 3800 60  0000 C CNN
@@
 $Comp
 L device:R R403
-U 1 1 5A0CA5F8
+U 1 1 5A369CF1
 P 3950 2700
 F 0 "R403" V 4050 2700 50  0000 C CNN
@@
 $Comp
 L device:R R402
-U 1 1 5A0CA5FF
+U 1 1 5A369CF4
 P 3950 3550
 F 0 "R402" V 3850 3550 50  0000 C CNN
@@
 $EndComp
 $Comp
-L power:GND #PWR0105
-U 1 1 5A0CA606
+L power:GND #PWR017
+U 1 1 5A369CF7
 P 3750 3950
-F 0 "#PWR0105" H 3750 3700 50  0001 C CNN
+F 0 "#PWR017" H 3750 3700 50  0001 C CNN
 F 1 "GND" H 3750 3800 50  0000 C CNN
 F 2 "" H 3750 3950 60  0000 C CNN
@@
 $Comp
 L Connector:Conn_01x04 P400
-U 1 1 5A0CA611
+U 1 1 5A369CF8
 P 5150 2950
 F 0 "P400" H 5150 3200 50  0000 C CNN
@@
 $Comp
 L device:C C408
-U 1 1 5A0CA61C
+U 1 1 5A369CFB
 P 2200 3400
 F 0 "C408" H 2225 3500 50  0000 L CNN
@@
 $EndComp
 $Comp
-L power:GND #PWR0106
-U 1 1 5A0CA623
+L power:GND #PWR018
+U 1 1 5A369CFE
 P 2050 3400
-F 0 "#PWR0106" H 2050 3150 50  0001 C CNN
+F 0 "#PWR018" H 2050 3150 50  0001 C CNN
 F 1 "GND" H 2050 3250 50  0000 C CNN
 F 2 "" H 2050 3400 60  0000 C CNN
@@
 $Comp
 L tmc2660:TMC2660 U400
-U 1 1 5A0CA62A
+U 1 1 5A369D02
 P 2950 2850
 F 0 "U400" H 2950 3150 60  0000 C CNN
@@
 $EndComp
 $Comp
-L power:GND #PWR0107
-U 1 1 5A0CA642
+L power:GND #PWR019
+U 1 1 5A369D06
 P 2250 3850
-F 0 "#PWR0107" H 2250 3600 50  0001 C CNN
+F 0 "#PWR019" H 2250 3600 50  0001 C CNN
 F 1 "GND" H 2250 3700 50  0000 C CNN
 F 2 "" H 2250 3850 60  0000 C CNN
@@
 NoConn ~ 2350 3250
 $Comp
-L power:GND #PWR0108
-U 1 1 5A0CA65B
+L power:GND #PWR020
+U 1 1 5A369D0C
 P 2250 2250
-F 0 "#PWR0108" H 2250 2000 50  0001 C CNN
+F 0 "#PWR020" H 2250 2000 50  0001 C CNN
 F 1 "GND" H 2250 2100 50  0000 C CNN
 F 2 "" H 2250 2250 60  0000 C CNN
@@
 $EndComp
 $Comp
-L power:GND #PWR0109
-U 1 1 5A0CA666
+L power:GND #PWR021
+U 1 1 5A369D0D
 P 2500 3800
-F 0 "#PWR0109" H 2500 3550 50  0001 C CNN
+F 0 "#PWR021" H 2500 3550 50  0001 C CNN
 F 1 "GND" H 2450 3650 50  0000 C CNN
 F 2 "" H 2500 3800 60  0000 C CNN
@@
 $Comp
 L device:R R400
-U 1 1 5A0CA66C
+U 1 1 5A369D10
 P 4400 3500
 F 0 "R400" H 4200 3500 50  0000 C CNN
@@
 $Comp
 L device:R R401
-U 1 1 5A0CA673
+U 1 1 5A369D13
 P 4400 2950
 F 0 "R401" H 4600 2900 50  0000 C CNN
@@
 $Comp
 L device:C_Small C401
-U 1 1 5A0CA67B
+U 1 1 5A369D18
 P 3800 2950
 F 0 "C401" H 3900 3000 50  0000 L CNN
@@
 Text Label 3500 2800 0    40   ~ 0
 BRA
-NoConn ~ 2350 3150
 Text Label 2000 2850 0    60   ~ 0
 STEP
@@
 $Comp
 L device:CP C407
-U 1 1 5A0CA6BD
+U 1 1 5A369D1C
 P 3500 1700
 F 0 "C407" H 3450 2000 50  0000 L CNN
@@
 Text HLabel 2050 2150 0    60   Input ~ 0
 ~EN
-$Comp
-L device:R J400
-U 1 1 5A0CA6C8
-P 1450 2350
-F 0 "J400" H 1550 2500 50  0000 C CNN
-F 1 "0R" V 1450 2350 50  0000 C CNN
-F 2 "Resistors_SMD:R_0603" V 1380 2350 30  0001 C CNN
-F 3 "" H 1450 2350 30  0000 C CNN
-	1    1450 2350
-	1    0    0    -1
-$EndComp
 Text HLabel 1250 2200 0    60   Input ~ 0
 START_MOSI
@@
 Text Label 4800 3150 0    60   ~ 0
 B2
-$Comp
-L Mechanical:Mounting_Hole M400
-U 1 1 5A0FBC47
-P 1250 4250
-F 0 "M400" H 1150 4400 50  0000 L CNN
-F 1 "Mount" H 1308 4279 50  0000 L CNN
-F 2 "Mounting_Holes:MountingHole_2.7mm_M2.5" H 1450 4250 50  0001 C CNN
-F 3 "~" H 1450 4250 50  0001 C CNN
-	1    1250 4250
-	1    0    0    -1
-$EndComp
-$Comp
-L Mechanical:Mounting_Hole_PAD M401
-U 1 1 5A0FBD0F
-P 1650 4300
-F 0 "M401" H 1550 4500 50  0000 L CNN
-F 1 "Mount" H 1708 4329 50  0000 L CNN
-F 2 "Mounting_Holes:MountingHole_2.7mm_M2.5_Pad" H 1850 4300 50  0001 C CNN
-F 3 "~" H 1850 4300 50  0001 C CNN
-	1    1650 4300
-	1    0    0    -1
-$EndComp
 Wire Wire Line
 	3050 1550 3050 1950
@@
 Wire Wire Line
 	1250 2200 1450 2200
-Connection ~ 1450 2500
 Wire Wire Line
 	3800 2700 3800 2850
@@
 Connection ~ 4250 2800
 $Comp
-L power:GND #PWR01
+L power:GND #PWR022
 U 1 1 5A17CB15
 P 4600 3200
-F 0 "#PWR01" H 4600 2950 50  0001 C CNN
+F 0 "#PWR022" H 4600 2950 50  0001 C CNN
 F 1 "GND" H 4600 3050 50  0000 C CNN
 F 2 "" H 4600 3200 60  0000 C CNN
@@
 Text Notes 4500 3750 0    51   ~ 0
 Sense Resistors alternatively\nalso with 100mOhm
-$Comp
-L power:GND #PWR?
-U 1 1 5A1C342B
-P 1650 4400
-F 0 "#PWR?" H 1650 4150 50  0001 C CNN
-F 1 "GND" H 1650 4250 50  0000 C CNN
-F 2 "" H 1650 4400 60  0000 C CNN
-F 3 "" H 1650 4400 60  0000 C CNN
-	1    1650 4400
-	1    0    0    -1
-$EndComp
 Wire Wire Line
 	3050 1550 3200 1550
@@
 Wire Wire Line
 	3750 3550 3800 3550
+Connection ~ 1450 2500
+$Comp
+L device:R J400
+U 1 1 5A369D20
+P 1450 2350
+F 0 "J400" H 1550 2500 50  0000 C CNN
+F 1 "0R" V 1450 2350 50  0000 C CNN
+F 2 "Resistors_SMD:R_0603" V 1380 2350 30  0001 C CNN
+F 3 "" H 1450 2350 30  0000 C CNN
+	1    1450 2350
+	1    0    0    -1
+$EndComp
+Text HLabel 1950 3150 0    60   Output ~ 0
+STALL
+Wire Wire Line
+	1950 3150 2350 3150
+Text Label 2000 3150 0    60   ~ 0
+STALL
 $EndSCHEMATC
