File: tmc2660/tmc2660-quad.sch (KiCad schematic (older format))
At the start: 5 parts, among them J1 Power, J2 DataIn, M0 Mount, M1 Mount

Commit message: Finished squished board
Parts:
- removed M0: Mount, Mounting_Holes:MountingHole_2.7mm_M2.5, symbol Mechanical:Mounting_Hole
- removed M1: Mount, Mounting_Holes:MountingHole_2.7mm_M2.5_Pad, symbol Mechanical:Mounting_Hole_PAD
- added D1: BAV70, TO_SOT_Packages_SMD:SOT-363_SC-70-6_Handsoldering, symbol diode:BAV70
- added J3: 10k, Resistors_SMD:R_0603, symbol device:R
Connections:
- net labels added: STALL
- wire segments 48 -> 75
- no-connect marks 1 -> 0
Changed lines of the file:
@@
 F10 "STEP" I L 4350 1950 60
 F11 "DIR" I L 4350 2050 60
+F12 "STALL" O L 4350 2350 60
 $EndSheet
 Text GLabel 4250 1650 0    60   Input ~ 0
@@
 F10 "STEP" I L 4350 4550 60
 F11 "DIR" I L 4350 4650 60
+F12 "STALL" O L 4350 4950 60
 $EndSheet
 Text GLabel 4250 4250 0    60   Input ~ 0
@@
 F10 "STEP" I L 4350 5850 60
 F11 "DIR" I L 4350 5950 60
+F12 "STALL" O L 4350 6250 60
 $EndSheet
 Text GLabel 4250 5550 0    60   Input ~ 0
@@
 	4350 2250 3850 2250
 Wire Wire Line
-	3850 2250 3850 6150
+	3850 2250 3850 2700
 Wire Wire Line
 	3850 6150 4350 6150
 Wire Wire Line
-	5350 2250 6050 2250
+	5350 2250 5500 2250
 Wire Wire Line
 	5500 6150 5350 6150
@@
 Connection ~ 5500 3550
 Wire Wire Line
-	5350 2150 6050 2150
-Wire Wire Line
-	5650 2150 5650 6050
+	5350 2150 5650 2150
+Wire Wire Line
+	5650 2150 5650 3450
 Wire Wire Line
 	5650 6050 5350 6050
@@
 	5350 5700 5850 5700
 Wire Wire Line
-	5850 1800 5850 5950
-Wire Wire Line
-	5350 1800 6050 1800
+	5850 1800 5850 3100
+Wire Wire Line
+	5350 1800 5850 1800
 Wire Wire Line
 	5350 3100 5850 3100
@@
 	1    0    0    -1
 $EndComp
-Wire Wire Line
-	2650 1800 2650 2000
-Connection ~ 2650 1900
 Text GLabel 3500 1600 2    60   Output ~ 0
 VMot
@@
 Wire Wire Line
 	2650 1600 3050 1600
-Connection ~ 2650 1600
-Wire Wire Line
-	5500 2250 5500 6150
+Wire Wire Line
+	5500 2250 5500 3550
 $Sheet
 S 4350 2850 1000 950
@@
 F10 "STEP" I L 4350 3250 60
 F11 "DIR" I L 4350 3350 60
+F12 "STALL" O L 4350 3650 60
 $EndSheet
 Wire Wire Line
@@
 Wire Wire Line
 	4200 5950 4350 5950
-Text GLabel 3800 2700 0    51   Input ~ 0
+Text GLabel 3700 2700 0    51   Input ~ 0
 ~ENABLE
-Wire Wire Line
-	3800 2700 3850 2700
 Connection ~ 3850 2700
 Text GLabel 2300 3250 0    47   Input ~ 0
@@
 Text GLabel 2800 3850 2    51   Input ~ 0
 DIR4
-NoConn ~ 2800 3250
 Wire Wire Line
 	5350 5950 5850 5950
 Connection ~ 5850 5700
-$Comp
-L Mechanical:Mounting_Hole M0
-U 1 1 5A1112B3
-P 2300 4550
-F 0 "M0" H 2250 4700 50  0000 L CNN
-F 1 "Mount" H 2200 4800 50  0000 L CNN
-F 2 "Mounting_Holes:MountingHole_2.7mm_M2.5" H 2500 4550 50  0001 C CNN
-F 3 "~" H 2500 4550 50  0001 C CNN
-	1    2300 4550
-	1    0    0    -1
-$EndComp
-$Comp
-L Mechanical:Mounting_Hole_PAD M1
-U 1 1 5A1112BA
-P 2700 4600
-F 0 "M1" H 2700 4800 50  0000 L CNN
-F 1 "Mount" H 2600 4900 50  0000 L CNN
-F 2 "Mounting_Holes:MountingHole_2.7mm_M2.5_Pad" H 2900 4600 50  0001 C CNN
-F 3 "~" H 2900 4600 50  0001 C CNN
-	1    2700 4600
-	1    0    0    -1
-$EndComp
 $Comp
 L device:Fuse F1
@@
 Text Label 2700 1600 0    60   ~ 0
 PowerIn
+Wire Wire Line
+	5500 4850 5500 6150
+Wire Wire Line
+	5500 3550 5500 4850
+Wire Wire Line
+	5650 4750 5650 6050
+Wire Wire Line
+	5650 3450 5650 4750
+Wire Wire Line
+	5850 3100 5850 4400
+Wire Wire Line
+	5850 4400 5850 5700
+Wire Wire Line
+	3850 4850 3850 6150
+Wire Wire Line
+	3850 3550 3850 4850
+Wire Wire Line
+	5850 1800 6050 1800
+Wire Wire Line
+	5650 2150 6050 2150
+Wire Wire Line
+	5500 2250 6050 2250
+Wire Wire Line
+	3850 2700 3850 3550
+Wire Wire Line
+	5850 5700 5850 5950
+Wire Wire Line
+	2650 1800 2650 2000
+Wire Wire Line
+	4250 6250 4350 6250
+Wire Wire Line
+	4050 6250 3775 6250
+Wire Wire Line
+	3775 6250 3775 4950
+Wire Wire Line
+	3700 2700 3850 2700
+Wire Wire Line
+	4250 4950 4350 4950
+Wire Wire Line
+	4250 3650 4350 3650
+Wire Wire Line
+	4250 2350 4350 2350
+Wire Wire Line
+	3775 2350 4050 2350
+Wire Wire Line
+	4050 3650 3775 3650
+Connection ~ 3775 3650
+Wire Wire Line
+	3775 3650 3775 2875
+Wire Wire Line
+	4050 4950 3775 4950
+Connection ~ 3775 4950
+Wire Wire Line
+	3775 4950 3775 3650
+Wire Wire Line
+	3775 6250 3775 6325
+Connection ~ 3775 6250
+$Comp
+L device:R J3
+U 1 1 5A361D50
+P 3775 6475
+F 0 "J3" H 3875 6625 50  0000 C CNN
+F 1 "10k" V 3775 6475 50  0000 C CNN
+F 2 "Resistors_SMD:R_0603" V 3705 6475 30  0001 C CNN
+F 3 "" H 3775 6475 30  0000 C CNN
+	1    3775 6475
+	1    0    0    -1
+$EndComp
 $Comp
 L power:GND #PWR02
-U 1 1 5A1C0ADE
-P 2700 4700
-F 0 "#PWR02" H 2700 4450 50  0001 C CNN
-F 1 "GND" V 2705 4572 50  0000 R CNN
-F 2 "" H 2700 4700 50  0001 C CNN
-F 3 "" H 2700 4700 50  0001 C CNN
-	1    2700 4700
-	1    0    0    -1
-$EndComp
+U 1 1 5A3641BC
+P 3775 6625
+F 0 "#PWR02" H 3775 6375 50  0001 C CNN
+F 1 "GND" H 3780 6452 50  0000 C CNN
+F 2 "" H 3775 6625 50  0001 C CNN
+F 3 "" H 3775 6625 50  0001 C CNN
+	1    3775 6625
+	1    0    0    -1
+$EndComp
+Text GLabel 3700 2875 0    60   Output ~ 0
+STALL
+Wire Wire Line
+	3700 2875 3775 2875
+Connection ~ 3775 2875
+Wire Wire Line
+	3775 2875 3775 2350
+Text GLabel 2800 3250 2    51   Input ~ 0
+STALL
+$Comp
+L diode:BAV70 D1
+U 4 1 5A3503F9
+P 4150 6250
+F 0 "D1" H 4150 6100 60  0000 C CNN
+F 1 "BAV70" H 4150 6175 60  0000 C CNN
+F 2 "TO_SOT_Packages_SMD:SOT-363_SC-70-6_Handsoldering" H 4150 6100 50  0001 C CNN
+F 3 "" H 4150 6150 60  0001 C CNN
+	4    4150 6250
+	1    0    0    -1
+$EndComp
+$Comp
+L diode:BAV70 D1
+U 3 1 5A351177
+P 4150 4950
+F 0 "D1" H 4150 4800 60  0000 C CNN
+F 1 "BAV70" H 4150 4875 60  0000 C CNN
+F 2 "TO_SOT_Packages_SMD:SOT-363_SC-70-6_Handsoldering" H 4150 4800 50  0001 C CNN
+F 3 "" H 4150 4850 60  0001 C CNN
+	3    4150 4950
+	1    0    0    -1
+$EndComp
+$Comp
+L diode:BAV70 D1
+U 2 1 5A35164F
+P 4150 2350
+F 0 "D1" H 4150 2200 60  0000 C CNN
+F 1 "BAV70" H 4150 2275 60  0000 C CNN
+F 2 "TO_SOT_Packages_SMD:SOT-363_SC-70-6_Handsoldering" H 4150 2200 50  0001 C CNN
+F 3 "" H 4150 2250 60  0001 C CNN
+	2    4150 2350
+	1    0    0    -1
+$EndComp
+$Comp
+L diode:BAV70 D1
+U 1 1 5A351CC9
+P 4150 3650
+F 0 "D1" H 4150 3500 60  0000 C CNN
+F 1 "BAV70" H 4150 3575 60  0000 C CNN
+F 2 "TO_SOT_Packages_SMD:SOT-363_SC-70-6_Handsoldering" H 4150 3500 50  0001 C CNN
+F 3 "" H 4150 3550 60  0001 C CNN
+	1    4150 3650
+	1    0    0    -1
+$EndComp

Commit message: Initial commit on gadgeteer port version
Parts:
- removed J2: DataIn, Quadrigotion:IDC_Header_SMD_16pins, symbol Connector:Conn_02x08_Odd_Even
- added J2: Gadgeteer S, Pin_Headers:Pin_Header_Straight_2x05_Pitch1.27mm_SMD, symbol Connector:Conn_02x05_Odd_Even
- added J4: Gadgeteer Y, Pin_Headers:Pin_Header_Straight_2x05_Pitch1.27mm_SMD, symbol Connector:Conn_02x05_Odd_Even
Connections:
- net labels added: +3V3
- wire segments 75 -> 86
- no-connect marks 0 -> 2
Changed lines of the file:
@@
-$EndComp
-$Comp
-L Connector:Conn_02x08_Odd_Even J2
-U 1 1 5A1095ED
-P 2500 3450
-F 0 "J2" H 2550 2825 50  0000 C CNN
-F 1 "DataIn" H 2550 2916 50  0000 C CNN
-F 2 "Quadrigotion:IDC_Header_SMD_16pins" H 2500 3450 50  0001 C CNN
-F 3 "~" H 2500 3450 50  0001 C CNN
-	1    2500 3450
-	1    0    0    -1
 $EndComp
 $Comp
 L power:GND #PWR0116
 U 1 1 5A109C26
-P 2300 3150
-F 0 "#PWR0116" H 2300 2900 50  0001 C CNN
-F 1 "GND" V 2305 3022 50  0000 R CNN
-F 2 "" H 2300 3150 50  0001 C CNN
-F 3 "" H 2300 3150 50  0001 C CNN
-	1    2300 3150
-	0    1    1    0
-$EndComp
-$Comp
-L power:VCC #PWR0115
-U 1 1 5A109EE9
-P 2800 3150
-F 0 "#PWR0115" H 2800 3000 50  0001 C CNN
-F 1 "VCC" V 2817 3278 50  0000 L CNN
-F 2 "" H 2800 3150 50  0001 C CNN
-F 3 "" H 2800 3150 50  0001 C CNN
-	1    2800 3150
-	0    1    1    0
+P 1825 3875
+F 0 "#PWR0116" H 1825 3625 50  0001 C CNN
+F 1 "GND" V 1830 3747 50  0000 R CNN
+F 2 "" H 1825 3875 50  0001 C CNN
+F 3 "" H 1825 3875 50  0001 C CNN
+	1    1825 3875
+	1    0    0    -1
 $EndComp
 Wire Wire Line
@@
 Connection ~ 5650 2150
 Connection ~ 5500 2250
-Text GLabel 2300 3350 0    51   Output ~ 0
+Text GLabel 1775 3625 2    51   Output ~ 0
 CS
-Text GLabel 2800 3350 2    51   Output ~ 0
+Text GLabel 1275 3825 0    51   Output ~ 0
 SCLK
-Text GLabel 2800 3450 2    51   Output ~ 0
+Text GLabel 1275 3725 0    51   Output ~ 0
 GLOBAL_MOSI
-Text GLabel 2300 3450 0    51   Input ~ 0
+Text GLabel 1775 3725 2    51   Input ~ 0
 GLOBAL_MISO
 $Comp
@@
 ~ENABLE
 Connection ~ 3850 2700
-Text GLabel 2300 3250 0    47   Input ~ 0
+Text GLabel 1275 3525 0    35   Input ~ 0
 ~ENABLE
-Text GLabel 2300 3550 0    51   Output ~ 0
+Text GLabel 1775 4675 2    51   Output ~ 0
 STEP1
-Text GLabel 2300 3650 0    51   Output ~ 0
+Text GLabel 1775 4475 2    51   Output ~ 0
 STEP2
-Text GLabel 2300 3750 0    51   Output ~ 0
+Text GLabel 1275 4575 0    51   Output ~ 0
 STEP3
-Text GLabel 2300 3850 0    51   Output ~ 0
+Text GLabel 1275 4775 0    51   Output ~ 0
 STEP4
-Text GLabel 2800 3550 2    51   Output ~ 0
+Text GLabel 1775 4575 2    51   Output ~ 0
 DIR1
-Text GLabel 2800 3650 2    51   Output ~ 0
+Text GLabel 1275 4475 0    51   Output ~ 0
 DIR2
-Text GLabel 2800 3750 2    51   Input ~ 0
+Text GLabel 1275 4675 0    51   Output ~ 0
 DIR3
-Text GLabel 2800 3850 2    51   Input ~ 0
+Text GLabel 1275 3625 0    51   Output ~ 0
 DIR4
 Wire Wire Line
@@
 Wire Wire Line
 	3775 2875 3775 2350
-Text GLabel 2800 3250 2    51   Input ~ 0
+Text GLabel 1775 3525 2    51   Input ~ 0
 STALL
 $Comp
@@
 	1    0    0    -1
 $EndComp
+$Comp
+L power:VCC #PWR0115
+U 1 1 5A109EE9
+P 700 2150
+F 0 "#PWR0115" H 700 2000 50  0001 C CNN
+F 1 "VCC" V 717 2278 50  0000 L CNN
+F 2 "" H 700 2150 50  0001 C CNN
+F 3 "" H 700 2150 50  0001 C CNN
+	1    700  2150
+	1    0    0    -1
+$EndComp
+$Comp
+L power:+3V3 #PWR034
+U 1 1 5A443542
+P 900 2150
+F 0 "#PWR034" H 900 2000 50  0001 C CNN
+F 1 "+3V3" H 915 2323 50  0000 C CNN
+F 2 "" H 900 2150 50  0001 C CNN
+F 3 "" H 900 2150 50  0001 C CNN
+	1    900  2150
+	1    0    0    -1
+$EndComp
+Wire Wire Line
+	700  2150 700  2200
+Wire Wire Line
+	700  2200 900  2200
+Wire Wire Line
+	900  2200 900  2150
+$Comp
+L power:+3V3 #PWR035
+U 1 1 5A4458CC
+P 1200 4300
+F 0 "#PWR035" H 1200 4150 50  0001 C CNN
+F 1 "+3V3" H 1215 4473 50  0000 C CNN
+F 2 "" H 1200 4300 50  0001 C CNN
+F 3 "" H 1200 4300 50  0001 C CNN
+	1    1200 4300
+	1    0    0    -1
+$EndComp
+$Comp
+L power:+3V3 #PWR036
+U 1 1 5A4601C3
+P 1200 3350
+F 0 "#PWR036" H 1200 3200 50  0001 C CNN
+F 1 "+3V3" H 1215 3523 50  0000 C CNN
+F 2 "" H 1200 3350 50  0001 C CNN
+F 3 "" H 1200 3350 50  0001 C CNN
+	1    1200 3350
+	1    0    0    -1
+$EndComp
+$Comp
+L Connector:Conn_02x05_Odd_Even J4
+U 1 1 5A47B1EE
+P 1475 4575
+F 0 "J4" H 1525 4992 50  0000 C CNN
+F 1 "Gadgeteer Y" H 1525 4901 50  0000 C CNN
+F 2 "Pin_Headers:Pin_Header_Straight_2x05_Pitch1.27mm_SMD" H 1475 4575 50  0001 C CNN
+F 3 "~" H 1475 4575 50  0001 C CNN
+	1    1475 4575
+	1    0    0    -1
+$EndComp
+Wire Wire Line
+	1200 4300 1200 4375
+Wire Wire Line
+	1200 4375 1275 4375
+NoConn ~ 1775 4375
+$Comp
+L power:GND #PWR037
+U 1 1 5A48035C
+P 1825 4825
+F 0 "#PWR037" H 1825 4575 50  0001 C CNN
+F 1 "GND" V 1830 4697 50  0000 R CNN
+F 2 "" H 1825 4825 50  0001 C CNN
+F 3 "" H 1825 4825 50  0001 C CNN
+	1    1825 4825
+	1    0    0    -1
+$EndComp
+Wire Wire Line
+	1775 4775 1825 4775
+Wire Wire Line
+	1825 4775 1825 4825
+$Comp
+L Connector:Conn_02x05_Odd_Even J2
+U 1 1 5A441394
+P 1475 3625
+F 0 "J2" H 1525 4042 50  0000 C CNN
+F 1 "Gadgeteer S" H 1525 3951 50  0000 C CNN
+F 2 "Pin_Headers:Pin_Header_Straight_2x05_Pitch1.27mm_SMD" H 1475 3625 50  0001 C CNN
+F 3 "~" H 1475 3625 50  0001 C CNN
+	1    1475 3625
+	1    0    0    -1
+$EndComp
+Wire Wire Line
+	1200 3350 1200 3425
+Wire Wire Line
+	1200 3425 1275 3425
+NoConn ~ 1775 3425
+Wire Wire Line
+	1775 3825 1825 3825
+Wire Wire Line
+	1825 3825 1825 3875
 $EndSCHEMATC
