File: tmc2660/tmc2660-quad.kicad_pcb (KiCad board)
At the start: 4 copper layers, 100 x 50 mm, 83 parts, among them J1 Power, J100 0R, J2 DataIn, J200 0R, J3 10k, J300 0R, J400 0R, M0 Mount, M1 Mount, M100 Mount, M101 Mount, M200 Mount, M201 Mount, M300 Mount, M301 Mount, P100 Motor, P200 Motor, P300 Motor, P400 Motor, U100 TMC2660, U200 TMC2660, U300 TMC2660, U400 TMC2660

Commit message: Initial commit on gadgeteer port version
Parts:
- added J4: Gadgeteer Y, Pin_Headers:Pin_Header_Straight_2x05_Pitch1.27mm_SMD, F.Cu at (124.4, 104.8)
- J2: value DataIn -> Gadgeteer S; footprint Quadrigotion:IDC_Header_SMD_16pins -> Pin_Headers:Pin_Header_Straight_2x05_Pitch1.27mm_SMD
- REF***: moved to B.Cu
- moved REF*** 89.3 mm to (147.8, 96.2), turned to 180 degrees
- moved G*** 5.65 mm to (147.5, 104.5)
- moved J3 3.13 mm to (107.4, 107.9), turned to 90 degrees
- moved J2 2.50 mm to (112.5, 104.8), turned to 270 degrees
- moved D1 1.35 mm to (107.3, 97.6)
Connections:
- C106 pad 1: VCC -> +3V3
- C206 pad 1: VCC -> +3V3
- C306 pad 1: VCC -> +3V3
- C406 pad 1: VCC -> +3V3
- J1 pad 4: GND -> Net-(J1-Pad4)
- J2 pad 1: GND -> +3V3
- J2 pad 10: DIR1 -> GND
- J2 pad 2: VCC -> Net-(J2-Pad2)
- J2 pad 5: CS -> DIR4
- J2 pad 6: SCLK -> CS
- J2 pad 7: GLOBAL_MISO -> GLOBAL_MOSI
- J2 pad 8: GLOBAL_MOSI -> GLOBAL_MISO
- J2 pad 9: STEP1 -> SCLK
- U100 pad 40: VCC -> +3V3
- U200 pad 40: VCC -> +3V3
- U300 pad 40: VCC -> +3V3
- U400 pad 40: VCC -> +3V3
Routing:
- net +3V3: track 0.00 -> 83.9 mm, vias 0 -> 7
- net VCC: track 66.7 -> 0.00 mm, vias 6 -> 0
- net DIR4: track 142.5 -> 120.5 mm
- net STEP4: track 143.7 -> 127.5 mm
- net GLOBAL_MISO: track 87.9 -> 73.5 mm
- net GLOBAL_MOSI: track 155.7 -> 144.0 mm
- net STALL: track 19.5 -> 30.9 mm, vias 0 -> 1
- net SCLK: track 147.9 -> 136.9 mm
- net DIR3: track 117.6 -> 109.2 mm
- net STEP3: track 118.6 -> 111.2 mm
- net CS: track 159.7 -> 152.4 mm
- net ~ENABLE: track 148.2 -> 143.8 mm
- net DIR2: track 92.3 -> 89.1 mm
- net GND: track 80.3 -> 83.1 mm, vias 92 -> 88
- net STEP1: track 68.0 -> 65.3 mm
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- added copper zone on In2.Cu, net +3V3
- removed copper zone on In2.Cu, net VCC
Other:
- board text added: "2017 Mikkel Jeppesen"
- board text added: "git.io/quadrigotion-duckle Multi Motor Driver"
- board text removed: "%%gitversion%%"
- board text removed: "MO"
- board text removed: "NC"
- board text removed: "S2 D2"
- board text removed: "S3 D3"
- board text removed: "S4 D4"
- board text removed: "http://qaudrigotion.org/ Multi Motor Driver"
- board text removed: "https://github.com/hzeller/quadrigotion"

Commit message: Added renders
Parts:
- removed the REF** at (262.2, 57.9)
Routing:
- net +3V3: track 83.9 -> 82.7 mm
Other:
- board text removed: "D2"
- board text removed: "D3"
- board text removed: "D4"
- board text removed: "MI"
- board text removed: "MOSI"
- board text removed: "N/C"
- board text removed: "S1"
- board text removed: "S2"
- board text removed: "S3"
- board text removed: "S4"
- board text removed: "SCLK"
- board text removed: "VCC"
- board text removed: "~CS"
- board text removed: "~EN"
Changed lines of the file:
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@@
   (general
     (thickness 1.6)
-    (drawings 36)
-    (tracks 1413)
+    (drawings 22)
+    (tracks 1414)
     (zones 0)
-    (modules 84)
+    (modules 83)
     (nets 73)
   )
@@
   )
   (setup
-    (last_trace_width 0.2)
+    (last_trace_width 0.6)
     (user_trace_width 0.2)
     (user_trace_width 0.3)
@@
     (user_trace_width 1.2)
     (trace_clearance 0.1778)
-    (zone_clearance 0.4)
+    (zone_clearance 0.3)
     (zone_45_only no)
     (trace_min 0.2)
@@
     (tags "Surface mounted pin header SMD 2x05 1.27mm double row")
     (attr smd)
-    (fp_text reference J4 (at 0 -4.235 270) (layer F.SilkS)
+    (fp_text reference J4 (at 0 -4.235 270) (layer F.SilkS) hide
       (effects (font (size 1 1) (thickness 0.15)))
     )
-    (fp_text value "Gadgeteer Y" (at 0 4.235 270) (layer F.Fab)
+    (fp_text value "Gadgeteer Y" (at 0.15 4.7 270) (layer F.SilkS)
       (effects (font (size 1 1) (thickness 0.15)))
     )
@@
     (tags "Surface mounted pin header SMD 2x05 1.27mm double row")
     (attr smd)
-    (fp_text reference J2 (at 0 -4.235 270) (layer F.SilkS)
+    (fp_text reference J2 (at 0 -4.235 270) (layer F.SilkS) hide
       (effects (font (size 1 1) (thickness 0.15)))
     )
-    (fp_text value "Gadgeteer S" (at 0 4.235 270) (layer F.Fab)
+    (fp_text value "Gadgeteer S" (at 0.05 -5.5 270) (layer F.SilkS)
       (effects (font (size 1 1) (thickness 0.15)))
     )
@@
     (zone_connect 2)
     (attr virtual)
-    (fp_text reference M1 (at 0 -3.7) (layer F.SilkS)
+    (fp_text reference M1 (at 0 -3.7) (layer F.SilkS) hide
       (effects (font (size 1 1) (thickness 0.15)))
     )
@@
     (zone_connect 2)
     (attr virtual)
-    (fp_text reference M201 (at -0.079 3.709) (layer F.SilkS)
+    (fp_text reference M201 (at -0.079 3.709) (layer F.SilkS) hide
       (effects (font (size 1 1) (thickness 0.15)))
     )
@@
     (zone_connect 2)
     (attr virtual)
-    (fp_text reference M101 (at -0.079 3.709) (layer F.SilkS)
+    (fp_text reference M101 (at -0.079 3.709) (layer F.SilkS) hide
       (effects (font (size 1 1) (thickness 0.15)))
     )
@@
     (zone_connect 2)
     (attr virtual)
-    (fp_text reference M301 (at -0.079 3.709) (layer F.SilkS)
+    (fp_text reference M301 (at -0.079 3.709) (layer F.SilkS) hide
       (effects (font (size 1 1) (thickness 0.15)))
     )
@@
     )
   )
-  (module Fiducials:Fiducial_0.5mm_Dia_1mm_Outer (layer F.Cu)
-    (at 262.2155 57.87)
-    (descr "Circular Fiducial, 0.5mm bare copper top; 1mm keepout (Level C)")
-    (tags marker)
-    (attr virtual)
-    (fp_text reference REF** (at 0 -1.5) (layer F.SilkS) hide
-      (effects (font (size 1 1) (thickness 0.15)))
-    )
-    (fp_text value Fiducial_0.5mm_Dia_1mm_Outer (at 0 1.5) (layer F.Fab) hide
-      (effects (font (size 1 1) (thickness 0.15)))
-    )
-    (fp_circle (center 0 0) (end 0.75 0) (layer F.CrtYd) (width 0.05))
-    (fp_text user %R (at 0 0) (layer F.Fab)
-      (effects (font (size 0.2 0.2) (thickness 0.04)))
-    )
-    (fp_circle (center 0 0) (end 0.5 0) (layer F.Fab) (width 0.1))
-    (pad ~ smd circle (at 0 0) (size 0.5 0.5) (layers F.Cu F.Mask)
-      (solder_mask_margin 0.25) (clearance 0.25))
-  )
   (module Symbols:OSHW-Symbol_6.7x6mm_SilkScreen locked (layer B.Cu)
     (at 147.75 96.25 180)
@@
     (tags "resistor 0603")
     (attr smd)
-    (fp_text reference J3 (at 0 -1.45 90) (layer F.SilkS)
+    (fp_text reference J3 (at 0 -1.45 90) (layer F.SilkS) hide
       (effects (font (size 1 1) (thickness 0.15)))
     )
@@
       (xy 1.961326 -4.735749) (xy 2.887919 -4.58736)) (layer F.Mask) (width 0.01))
   )
+  (gr_text 1 (at 116.9 102.4) (layer F.SilkS)
+    (effects (font (size 1 1) (thickness 0.25)))
+  )
+  (gr_text 1 (at 128.8 102.4) (layer F.SilkS)
+    (effects (font (size 1 1) (thickness 0.25)))
+  )
   (gr_text "2017\nMikkel Jeppesen" (at 134.25 107.25) (layer F.SilkS)
     (effects (font (size 1 1) (thickness 0.2)))
   )
-  (gr_text S4 (at 16.8935 38.1005) (layer B.SilkS)
-    (effects (font (size 1.2 1.2) (thickness 0.2)) (justify left mirror))
-  )
   (gr_line (start 199.4655 109.87) (end 99.4655 109.87) (layer Edge.Cuts) (width 0.1))
   (dimension 50 (width 0.3) (layer Cmts.User)
@@
     (effects (font (size 2.2 2.2) (thickness 0.4)) (justify mirror))
   )
-  (gr_text VCC (at 22.3935 20.3205) (layer B.SilkS)
-    (effects (font (size 1.2 1.2) (thickness 0.2)) (justify right mirror))
-  )
-  (gr_text N/C (at 22.3935 22.8605) (layer B.SilkS)
-    (effects (font (size 1.2 1.2) (thickness 0.2)) (justify right mirror))
-  )
-  (gr_text SCLK (at 22.3935 25.4005) (layer B.SilkS)
-    (effects (font (size 1.2 1.2) (thickness 0.2)) (justify right mirror))
-  )
-  (gr_text MOSI (at 22.3935 27.9405) (layer B.SilkS)
-    (effects (font (size 1.2 1.2) (thickness 0.2)) (justify right mirror))
-  )
-  (gr_text D1 (at 22.3935 30.4805) (layer B.SilkS)
-    (effects (font (size 1.2 1.2) (thickness 0.2)) (justify right mirror))
-  )
-  (gr_text D2 (at 22.3935 33.0205) (layer B.SilkS)
-    (effects (font (size 1.2 1.2) (thickness 0.2)) (justify right mirror))
-  )
-  (gr_text D3 (at 22.3935 35.5605) (layer B.SilkS)
-    (effects (font (size 1.2 1.2) (thickness 0.2)) (justify right mirror))
-  )
-  (gr_text D4 (at 22.3935 38.1005) (layer B.SilkS)
-    (effects (font (size 1.2 1.2) (thickness 0.2)) (justify right mirror))
-  )
-  (gr_text S3 (at 16.8935 35.5605) (layer B.SilkS)
-    (effects (font (size 1.2 1.2) (thickness 0.2)) (justify left mirror))
-  )
-  (gr_text S2 (at 16.8935 33.0205) (layer B.SilkS)
-    (effects (font (size 1.2 1.2) (thickness 0.2)) (justify left mirror))
-  )
-  (gr_text S1 (at 16.8935 30.4805) (layer B.SilkS)
-    (effects (font (size 1.2 1.2) (thickness 0.2)) (justify left mirror))
-  )
-  (gr_text MI (at 16.8935 27.9405) (layer B.SilkS)
-    (effects (font (size 1.2 1.2) (thickness 0.2)) (justify left mirror))
-  )
-  (gr_text ~CS (at 16.8935 25.4005) (layer B.SilkS)
-    (effects (font (size 1.2 1.2) (thickness 0.2)) (justify left mirror))
-  )
-  (gr_text ~EN (at 16.8935 22.9875) (layer B.SilkS)
-    (effects (font (size 1.2 1.2) (thickness 0.2)) (justify left mirror))
-  )
-  (gr_text GND (at 17.389 18.2885) (layer B.SilkS)
-    (effects (font (size 1.2 1.2) (thickness 0.2)) (justify mirror))
-  )
   (gr_text " Z\n" (at 103.159 62.7325) (layer In2.Cu)
     (effects (font (size 3 3) (thickness 0.4)))
@@
   (segment (start 108.65 85.95) (end 106.55 88.05) (width 0.2) (layer In2.Cu) (net 68))
   (segment (start 106.55 94.05) (end 107.3 94.8) (width 0.2) (layer In2.Cu) (net 68))
+  (segment (start 118.85 99.6) (end 117.85 99.6) (width 0.6) (layer F.Cu) (net 69))
+  (segment (start 117.85 99.6) (end 117.25 99) (width 0.6) (layer F.Cu) (net 69))
+  (via (at 117.25 99) (size 0.8) (drill 0.4) (layers F.Cu B.Cu) (net 69))
+  (segment (start 120.65 99.6) (end 118.85 99.6) (width 0.6) (layer F.Cu) (net 69))
   (segment (start 117.25 99) (end 117.25 96.249104) (width 0.8) (layer In2.Cu) (net 69))
   (segment (start 117.25 96.249104) (end 118.4155 95.083604) (width 0.8) (layer In2.Cu) (net 69))
   (segment (start 118.4155 95.083604) (end 118.4155 88.52) (width 0.8) (layer In2.Cu) (net 69))
-  (segment (start 117.25 99) (end 119.25 101) (width 0.6) (layer In2.Cu) (net 69))
   (segment (start 116.25 101) (end 116.25 100) (width 0.6) (layer In2.Cu) (net 69))
   (segment (start 116.25 100) (end 117.25 99) (width 0.6) (layer In2.Cu) (net 69))
   (segment (start 121.5 99.6) (end 120.65 99.6) (width 0.6) (layer F.Cu) (net 69))
-  (segment (start 120.65 99.6) (end 119.25 101) (width 0.6) (layer F.Cu) (net 69))
   (segment (start 126.5 99.6) (end 121.5 99.6) (width 0.6) (layer F.Cu) (net 69))
-  (via (at 119.25 101) (size 0.8) (drill 0.4) (layers F.Cu B.Cu) (net 69))
   (segment (start 115.75 100.5) (end 116 100.75) (width 0.6) (layer F.Cu) (net 69))
   (segment (start 115.04 100.71) (end 115.25 100.5) (width 0.6) (layer F.Cu) (net 69))
@@
     )
   )
-  (zone (net 1) (net_name GND) (layer F.Cu) (hatch edge 0.508)
-    (connect_pads (clearance 0.3))
-    (min_thickness 0.254)
-    (fill yes (arc_segments 16) (thermal_gap 0.3) (thermal_bridge_width 0.508))
-    (polygon
-      (pts
-        (xy 201.0335 87.541) (xy 102.854283 87.541) (xy 102.9 93.85) (xy 164.2 93.75) (xy 164.2 109.85)
-        (xy 99.45 109.85) (xy 99.45 86.85) (xy 99.466362 86.850481) (xy 99.5 59.9) (xy 201.0335 59.601)
-      )
-    )
-  )
   (zone (net 2) (net_name VMot) (layer B.Cu) (hatch edge 0.508)
     (priority 2)
@@
       )
     )
+  )
+  (zone (net 1) (net_name GND) (layer F.Cu) (hatch edge 0.508)
+    (connect_pads thru_hole_only (clearance 0.3))
+    (min_thickness 0.254)
+    (fill yes (arc_segments 16) (thermal_gap 0.3) (thermal_bridge_width 0.508))
+    (polygon
+      (pts
+        (xy 201.0335 87.541) (xy 102.854283 87.541) (xy 99.5 87.5) (xy 99.5 59.9) (xy 201.0335 59.601)
+      )
+    )
+  )
+  (zone (net 1) (net_name GND) (layer F.Cu) (hatch edge 0.508)
+    (connect_pads (clearance 0.3))
+    (min_thickness 0.254)
+    (fill yes (arc_segments 16) (thermal_gap 0.3) (thermal_bridge_width 0.508))
+    (polygon
+      (pts
+        (xy 99.5 87) (xy 99.5 109.9) (xy 164.2 109.9) (xy 164.2 93.8) (xy 102.9 93.9)
+        (xy 102.9 87)
+      )
+    )
